File: boardSCH/PS4-sequencer.kicad_pcb (KiCad board)
At the start: 2 copper layers, 79.3 x 48 mm, 7 parts

Commit message: 1
Parts:
- removed the M1 at (127.9, 90.6)
- added ?: , , F.Cu at (122.2, 95.5)
- added ?: , , F.Cu at (123.1, 105.0)
- added ?: , , F.Cu at (124.5, 82.0)
- added ?: , , F.Cu at (131.0, 93.5)
- added ?: , , F.Cu at (167.0, 101.0)
- added ?: , , F.Cu at (154.5, 98.5)
- added ?: , , F.Cu at (126.8, 86.0)
- added ?: , , F.Cu at (154.5, 103.5)
- added ?: , , F.Cu at (123.3, 95.5)
- added ?: , , F.Cu at (136.0, 109.5)
- added ?: , , F.Cu at (124.5, 84.5)
- added ?: , , F.Cu at (121.0, 95.5)
- added ?: , , F.Cu at (154.5, 101.0)
- added ?: , , F.Cu at (119.8, 95.5)
- added ?: , , F.Cu at (110.5, 118.5)
- added ?: , , F.Cu at (125.0, 95.5)
- added ?: , , F.Cu at (129.0, 86.0)
- added ?: , , F.Cu at (127.0, 95.5)
- added ?: , , F.Cu at (130.3, 83.3)
- added ?: , , F.Cu at (115.0, 106.0)
- added ?: , , F.Cu at (170.0, 101.0)
- added ?: , , F.Cu at (129.5, 95.5)
- added ?: , , F.Cu at (162.0, 101.0)
- added ?: , , F.Cu at (137.0, 114.0)
- added ?: , , F.Cu at (154.5, 96.0)
- added ?: , , F.Cu at (176.5, 83.5)
- added ?: , , F.Cu at (173.5, 104.0)
- added ?: , , F.Cu at (165.0, 101.0)
- added ?: , , F.Cu at (177.5, 104.0)
- added G***: LOGO, ZoeDraw:zoeSilk, B.Cu at (148.2, 119.5)
- added J1: USB_A, digikey-footprints:USB_A_Female_UE27AC54100, B.Cu at (166.0, 91.8)
- added REF**: TestPoint_Pad_1.5x1.5mm, TestPoint:TestPoint_Pad_1.5x1.5mm, B.Cu at (159.5, 122.0)
- added REF**: TestPoint_Pad_1.5x1.5mm, TestPoint:TestPoint_Pad_1.5x1.5mm, B.Cu at (159.5, 119.0)
- added REF**: TestPoint_Pad_1.5x1.5mm, TestPoint:TestPoint_Pad_1.5x1.5mm, B.Cu at (159.5, 116.0)
- added t1: ~, TestPoint:TestPoint_Pad_1.5x1.5mm, B.Cu at (113.0, 98.0)
- added t2: ~, TestPoint:TestPoint_Pad_1.5x1.5mm, B.Cu at (113.0, 100.5)
- RZ1: moved to B.Cu
- moved RZ1 10.1 mm to (151.5, 106.1), turned to 180 degrees
Connections:
- RZ1 pad 1: unconnected-(RZ1-GP0-Pad1) -> Net-(J1-D+)
- RZ1 pad 10: unconnected-(RZ1-GP9-Pad10) -> /m5
- RZ1 pad 11: unconnected-(RZ1-GP10-Pad11) -> /m4
- RZ1 pad 12: unconnected-(RZ1-GP11-Pad12) -> GND
- RZ1 pad 13: unconnected-(RZ1-GP12-Pad13) -> GND
- RZ1 pad 14: unconnected-(RZ1-GP13-Pad14) -> /m15
- RZ1 pad 15: unconnected-(RZ1-GP14-Pad15) -> /m3
- RZ1 pad 16: unconnected-(RZ1-GP15-Pad16) -> /m13
- RZ1 pad 17: /PS_BUTTON -> /m18
- RZ1 pad 18: unconnected-(RZ1-GP27-Pad18) -> /m19
- RZ1 pad 19: unconnected-(RZ1-GP28-Pad19) -> Net-(RZ1-GP28)
- RZ1 pad 2: unconnected-(RZ1-GP1-Pad2) -> Net-(J1-D-)
- RZ1 pad 20: unconnected-(RZ1-GP29-Pad20) -> Net-(RZ1-GP29)
- RZ1 pad 3: Net-(RZ1-GP2) -> /m11
- RZ1 pad 4: Net-(RZ1-GP3) -> /m14
- RZ1 pad 5: unconnected-(RZ1-GP4-Pad5) -> /m12
- RZ1 pad 6: unconnected-(RZ1-GP5-Pad6) -> /PS_BUTTON
- RZ1 pad 7: unconnected-(RZ1-GP6-Pad7) -> /m9
- RZ1 pad 8: unconnected-(RZ1-GP7-Pad8) -> /m7
- RZ1 pad 9: unconnected-(RZ1-GP8-Pad9) -> /m6
- ShareLol1 pad 2: Net-(RZ1-GP3) -> Net-(RZ1-GP28)
- ShareLol1 pad 3: Net-(RZ1-GP3) -> Net-(RZ1-GP28)
- Start1 pad 1: GND -> Net-(RZ1-GP29)
- Start1 pad 2: Net-(RZ1-GP2) -> GND
- Start1 pad 3: Net-(RZ1-GP2) -> GND
- Start1 pad 4: GND -> Net-(RZ1-GP29)
- U1 pad B1A: unconnected-(U1-PadB1A) -> GND
- U1 pad B1B: unconnected-(U1-PadB1B) -> GND
- U1 pad B2A: unconnected-(U1-PadB2A) -> GND
- U1 pad B2B: unconnected-(U1-PadB2B) -> GND
- U1 pad H1: unconnected-(U1-H+-PadH1) -> Net-(U1-H+)
- U1 pad H3: unconnected-(U1-H--PadH3) -> GND
- U1 pad MOUNT1: unconnected-(U1-GND@1-PadMOUNT1) -> GND
- U1 pad MOUNT2: unconnected-(U1-GND@2-PadMOUNT2) -> GND
- U1 pad MOUNT3: unconnected-(U1-GND@3-PadMOUNT3) -> GND
- U1 pad MOUNT4: unconnected-(U1-GND@4-PadMOUNT4) -> GND
- U1 pad V1: unconnected-(U1-V+-PadV1) -> Net-(U1-H+)
- U1 pad V3: unconnected-(U1-V--PadV3) -> GND
- U2 pad B1A: unconnected-(U2-PadB1A) -> GND
- U2 pad B1B: unconnected-(U2-PadB1B) -> GND
- U2 pad B2A: unconnected-(U2-PadB2A) -> GND
- U2 pad B2B: unconnected-(U2-PadB2B) -> GND
- U2 pad H1: unconnected-(U2-H+-PadH1) -> Net-(U1-H+)
- U2 pad H3: unconnected-(U2-H--PadH3) -> GND
- U2 pad MOUNT1: unconnected-(U2-GND@1-PadMOUNT1) -> GND
- U2 pad MOUNT2: unconnected-(U2-GND@2-PadMOUNT2) -> GND
- U2 pad MOUNT3: unconnected-(U2-GND@3-PadMOUNT3) -> GND
- U2 pad MOUNT4: unconnected-(U2-GND@4-PadMOUNT4) -> GND
- U2 pad V1: unconnected-(U2-V+-PadV1) -> Net-(U1-H+)
- U2 pad V3: unconnected-(U2-V--PadV3) -> GND
Routing:
- net GND: track 0.00 -> 304.0 mm, vias 0 -> 5
- net Net-(U1-H+): track 0.00 -> 79.6 mm, vias 0 -> 2
- net /m3: track 0.00 -> 57.9 mm, vias 0 -> 1
- net Net-(J1-D+): track 0.00 -> 49.7 mm, vias 0 -> 2
- net Net-(J1-D-): track 0.00 -> 45.2 mm, vias 0 -> 1
- net Net-(RZ1-GP29): track 0.00 -> 37.1 mm, vias 0 -> 2
- net Net-(RZ1-GP28): track 0.00 -> 35.0 mm, vias 0 -> 2
- net /m4: track 0.00 -> 35.0 mm, vias 0 -> 1
- net /m13: track 0.00 -> 29.7 mm, vias 0 -> 1
- net /m15: track 0.00 -> 29.1 mm, vias 0 -> 1
- net /m5: track 0.00 -> 26.0 mm, vias 0 -> 1
- net /VCC: track 0.00 -> 24.8 mm, vias 0 -> 2
- net /m18: track 0.00 -> 21.5 mm, vias 0 -> 1
- net /m19: track 0.00 -> 20.9 mm, vias 0 -> 1
- net /m6: track 0.00 -> 17.7 mm, vias 0 -> 1
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Other:
- outline, holes or cut-outs redrawn
- board text added: "+"
- board text added: "11"
- board text added: "13"
- board text added: "18"
- board text added: "19"
- board text added: "3"
- board text added: "4"
- board text added: "9"
- board text added: "GND"
- board text added: "GP2040 board Fotten 2025 Rev 1"
- board text added: "Sharelol"
- board text added: "Start"
- board text added: "VCC"
- board text added: "d+"
- board text added: "d-"
- board text removed: "GP2040 board Fotten 2025 Rev1"
