File: boardSCH/PS4-sequencer.kicad_sch (KiCad schematic)
At the start: 7 parts, among them J1 USB_A

Commit message: 1
Parts:
- added t1, t2: ~, TestPoint:TestPoint_Pad_1.5x1.5mm, symbol Connector:TestPoint
Connections:
- net GND: now also RZ1.12 (GP11), RZ1.13 (GP12), Start1.2 (1), Start1.3 (1), U1.B1A, U1.B1B, U1.B2A, U1.B2B, U1.H3 (H-), U1.MOUNT1 (GND@1), U1.MOUNT2 (GND@2), U1.MOUNT3 (GND@3), U1.MOUNT4 (GND@4), U1.V3 (V-), U2.B1A, U2.B1B, U2.B2A, U2.B2B, U2.H3 (H-), U2.MOUNT1 (GND@1), U2.MOUNT2 (GND@2), U2.MOUNT3 (GND@3), U2.MOUNT4 (GND@4), U2.V3 (V-); no longer Start1.1 (2), Start1.4 (2)
- net PS_BUTTON: now also RZ1.6 (GP5); no longer RZ1.17 (GP26)
- net m1: now also t1.1
- net m11: now also RZ1.3 (GP2)
- net m12: now also RZ1.5 (GP4)
- net m13: now also RZ1.16 (GP15)
- net m14: now also RZ1.4 (GP3)
- net m15: now also RZ1.14 (GP13)
- net m18: now also RZ1.17 (GP26)
- net m19: now also RZ1.18 (GP27)
- net m2: now also t2.1
- net m3: now also RZ1.15 (GP14)
- net m4: now also RZ1.11 (GP10)
- net m5: now also RZ1.10 (GP9)
- net m6: now also RZ1.9 (GP8)
- net m7: now also RZ1.8 (GP7)
- net m9: now also RZ1.7 (GP6)
- net at RZ1.19 (GP28): now also ShareLol1.2 (1), ShareLol1.3 (1)
- net at RZ1.20 (GP29): now also Start1.1 (2), Start1.4 (2)
- net at U1.H1 (H+): now also U1.V1 (V+), U2.H1 (H+), U2.V1 (V+)
Other:
- moved on the sheet: M1, ShareLol1, Start1
